Commit message: initial commit

File: src/rover_description/robot/parts/base/base.urdf.xacro (robot description, xacro)
@@ -1,3 +1,22 @@
 <?xml version="1.0"?>
 <robot xmlns:xacro="http://www.ros.org/wiki/xacro">
+  <xacro:macro name="base_v0" params="parent *joint_origin">
+    <joint name="base_link_joint" type="fixed">
+      <xacro:insert_block name="joint_origin"/>
+      <parent link="${parent}"/>
+      <child link="base_link"/>
+    </joint>
+    <link name="base_link">
+      <visual>
+        <geometry>
+          <mesh filename="package://rover_description/meshes/STL/base/main_frame.stl"/>
+        </geometry>
+      </visual>
+      <collision>
+        <geometry>
+          <mesh filename="package://rover_description/meshes/STL/base/main_frame.stl"/>
+        </geometry>
+      </collision>
+    </link>
+  </xacro:macro>
 </robot>

File: src/rover_description/robot/parts/wheel/wheel.urdf.xacro (robot description, xacro)
@@ -1,3 +1,24 @@
 <?xml version="1.0"?>
 <robot xmlns:xacro="http://www.ros.org/wiki/xacro">
+    <xacro:macro name="wheel_v0" params="prefix parent *joint_origin *joint_axis">
+        <joint name="${prefix}_wheel_joint" type="continuous">
+            <xacro:insert_block name="joint_origin" />
+            <parent link="${parent}" />
+            <child link="${prefix}_wheel_link" />
+                <limit effort="1.5" velocity="20" />
+            <xacro:insert_block name="joint_axis"/>
+        </joint>
+        <link name="${prefix}_wheel_link">
+            <visual>
+                <geometry>
+                    <mesh filename="package://rover_description/meshes/STL/wheel/wheel_right.stl" />
+                </geometry>
+            </visual>
+            <collision>
+                <geometry>
+                    <mesh filename="package://rover_description/meshes/STL/wheel/wheel_right.stl" />
+                </geometry>
+            </collision>
+        </link>
+    </xacro:macro>
 </robot>

File: src/rover_description/robot/rover_main.urdf.xacro (robot description, xacro)
@@ -1,3 +1,30 @@
 <?xml version="1.0"?>
 <robot xmlns:xacro="http://www.ros.org/wiki/xacro" name="vision_robot">
+    <xacro:include filename="$(find rover_description)/robot/parts/base/base.urdf.xacro" />
+    <xacro:include filename="$(find rover_description)/robot/parts/wheel/wheel.urdf.xacro"/>
+    <link name="world" />
+    <xacro:base_v0 parent="world">
+        <joint_origin>
+            <origin xyz="5 0 0" rpy="0 0 0" />
+        </joint_origin>
+    </xacro:base_v0>
+    <!-- <link name="base_link">
+        <visual>
+            <geometry>
+                <mesh filename="package://rover_description/meshes/STL/base/main_frame.stl" />
+            </geometry>
+        </visual>
+    </link> -->
+    <xacro:wheel_v0 prefix="fr" parent="base_link">
+        <joint_origin>
+            <origin xyz="0 0 0" />
+        </joint_origin>
+        <axis xyz="0 0 0"/>
+    </xacro:wheel_v0>
+    <xacro:wheel_v0 prefix="fl" parent="base_link">
+        <joint_origin>
+            <origin value ="15 0 0"/>
+        </joint_origin>
+        <axis xyz="0 0 0" />
+    </xacro:wheel_v0>
 </robot>
